Commit message: update the aliengo usd with small and big Angel Limits

File: source/leggedloco_tasks/data/Robots/Unitree/Aliengo/aliengo_description/urdf/aliengo_bigAng.urdf (robot description, URDF)
Before this commit: robot aliengo, 31 links, 30 joints
Joints:
- joint FL_calf_joint: limit lower=-2.775 upper=-0.611 effort=55 velocity=15.89 -> lower=-2.775073510670984 upper=-0.6457718232379019 effort=44.4 velocity=15.89
- joint FL_hip_joint: limit lower=-0.873 upper=1.047 effort=44 velocity=20 -> lower=-1.2217304763960306 upper=1.2217304763960306 effort=35.278 velocity=20
- joint FL_thigh_joint: limit lower=-0.524 upper=3.927 effort=44 velocity=20 -> lower=-3.141592654 upper=4.71238898 effort=35.278 velocity=20
- joint FR_calf_joint: limit lower=-2.775 upper=-0.611 effort=55 velocity=15.89 -> lower=-2.775073510670984 upper=-0.6457718232379019 effort=44.4 velocity=15.89
- joint FR_hip_joint: limit lower=-0.873 upper=1.047 effort=44 velocity=20 -> lower=-1.2217304763960306 upper=1.2217304763960306 effort=35.278 velocity=20
- joint FR_thigh_joint: limit lower=-0.524 upper=3.927 effort=44 velocity=20 -> lower=-3.141592654 upper=4.71238898 effort=35.278 velocity=20
- joint RL_calf_joint: limit lower=-2.775 upper=-0.611 effort=55 velocity=15.89 -> lower=-2.775073510670984 upper=-0.6457718232379019 effort=44.4 velocity=15.89
- joint RL_hip_joint: limit lower=-0.873 upper=1.047 effort=44 velocity=20 -> lower=-1.2217304763960306 upper=1.2217304763960306 effort=35.278 velocity=20
- joint RL_thigh_joint: limit lower=-0.524 upper=3.927 effort=44 velocity=20 -> lower=-3.141592654 upper=4.71238898 effort=35.278 velocity=20
- joint RR_calf_joint: limit lower=-2.775 upper=-0.611 effort=55 velocity=15.89 -> lower=-2.775073510670984 upper=-0.6457718232379019 effort=44.4 velocity=15.89
- joint RR_hip_joint: limit lower=-0.873 upper=1.047 effort=44 velocity=20 -> lower=-1.2217304763960306 upper=1.2217304763960306 effort=35.278 velocity=20
- joint RR_thigh_joint: limit lower=-0.524 upper=3.927 effort=44 velocity=20 -> lower=-3.141592654 upper=4.71238898 effort=35.278 velocity=20
